File: KiCAD/driverDisplayLED.sch (KiCad schematic (older format))
At the start: 68 parts, among them J1 Conn_01x12_Male, J10 Conn_01x12_Male, J11 Conn_01x12_Male, J12 Conn_01x12_Male, J13 Conn_01x12_Male, J14 Conn_01x12_Male, J15 Conn_01x12_Male, J16 Conn_01x12_Male, J17 Conn_01x12_Male, J19 Conn_01x02_Female, J2 Conn_01x12_Male, J3 Conn_01x12_Male, J4 Conn_02x08_Counter_Clockwise, J5 Conn_01x12_Male, J6 Conn_01x12_Male, J7 Conn_01x12_Male, J8 Conn_01x12_Male, J9 Conn_01x12_Male, Q1 FDS4953, Q2 FDS4953, Q3 FDS4953, Q4 FDS4953, Q5 FDS4953, Q6 FDS4953, Q7 FDS4953, Q8 FDS4953, U1 74HC245, U10 74HC04, U2 74HC595, U3 74HC595, U4 74HC245, U5 74HC138D, U7 74HC595, U8 74HC595, U9 74HC138D

Commit message: Datasheets folder
Parts:
- L1, L2, L3, L4, L5, L6, L7, L8: symbol myLedMatrix:LedMatrix_M -> driverDisplayLED-rescue:LedMatrix_M-myLedMatrix
Connections:
- net GND: now also U1.2 (A0)
- no-connect marks 12 -> 11
Changed lines of the file:
@@
 	13750 5325 13750 4975
 Connection ~ 13750 5325
-NoConn ~ 1725 9400
 Wire Wire Line
 	1125 9600 1125 10725
@@
 	1875 3000 1875 3400
 $Comp
-L myLedMatrix:LedMatrix_M L8
+L driverDisplayLED-rescue:LedMatrix_M-myLedMatrix L8
 U 1 1 65EB8954
 P 7525 6400
@@
 $EndComp
 $Comp
-L myLedMatrix:LedMatrix_M L6
+L driverDisplayLED-rescue:LedMatrix_M-myLedMatrix L6
 U 1 1 65EB88FC
 P 5800 6400
@@
 $EndComp
 $Comp
-L myLedMatrix:LedMatrix_M L4
+L driverDisplayLED-rescue:LedMatrix_M-myLedMatrix L4
 U 1 1 65BA6083
 P 4000 6400
@@
 $EndComp
 $Comp
-L myLedMatrix:LedMatrix_M L2
+L driverDisplayLED-rescue:LedMatrix_M-myLedMatrix L2
 U 1 1 61F8FA0C
 P 2225 6400
@@
 $EndComp
 $Comp
-L myLedMatrix:LedMatrix_M L7
+L driverDisplayLED-rescue:LedMatrix_M-myLedMatrix L7
 U 1 1 6453BC83
 P 7525 3975
@@
 $EndComp
 $Comp
-L myLedMatrix:LedMatrix_M L5
+L driverDisplayLED-rescue:LedMatrix_M-myLedMatrix L5
 U 1 1 63DACAC0
 P 5775 3975
@@
 $EndComp
 $Comp
-L myLedMatrix:LedMatrix_M L3
+L driverDisplayLED-rescue:LedMatrix_M-myLedMatrix L3
 U 1 1 6153BDC2
 P 4000 3975
@@
 $EndComp
 $Comp
-L myLedMatrix:LedMatrix_M L1
+L driverDisplayLED-rescue:LedMatrix_M-myLedMatrix L1
 U 1 1 5FAA9D97
 P 2225 3975
@@
 Wire Bus Line
 	18725 4575 20725 4575
+$Comp
+L power:GND #PWR?
+U 1 1 60B63B1A
+P 1500 9200
+F 0 "#PWR?" H 1500 8950 50  0001 C CNN
+F 1 "GND" H 1505 9027 50  0000 C CNN
+F 2 "" H 1500 9200 50  0001 C CNN
+F 3 "" H 1500 9200 50  0001 C CNN
+	1    1500 9200
+	1    0    0    -1
+$EndComp
+Wire Wire Line
+	1650 9400 1650 9100
+Wire Wire Line
+	1650 9100 1500 9100
+Wire Wire Line
+	1500 9100 1500 9200
 Wire Bus Line
 	9275 9750 9275 9850
@@
 Wire Bus Line
 	1850 2650 13350 2650
+Wire Wire Line
+	1725 9400 1650 9400
 $EndSCHEMATC
