File: KiCAD/driverDisplayLED.sch (KiCad schematic (older format))
At the start: 68 parts, among them J1 Conn_01x12_Male, J10 Conn_01x12_Male, J11 Conn_01x12_Male, J12 Conn_01x12_Male, J13 Conn_01x12_Male, J14 Conn_01x12_Male, J15 Conn_01x12_Male, J16 Conn_01x12_Male, J17 Conn_01x12_Male, J19 Conn_01x02_Female, J2 Conn_01x12_Male, J3 Conn_01x12_Male, J4 Conn_02x08_Counter_Clockwise, J5 Conn_01x12_Male, J6 Conn_01x12_Male, J7 Conn_01x12_Male, J8 Conn_01x12_Male, J9 Conn_01x12_Male, Q1 FDS4953, Q2 FDS4953, Q3 FDS4953, Q4 FDS4953, Q5 FDS4953, Q6 FDS4953, Q7 FDS4953, Q8 FDS4953, U1 74HC245, U10 74HC04, U2 74HC595, U3 74HC595, U4 74HC245, U5 74HC138D, U7 74HC595, U8 74HC595, U9 74HC138D

Commit message: inicio esquemáticos de la placa de control
Parts:
- R1: value R -> 0
- R2: value R -> 5.1K
- R3: value R -> 100K
Changed lines of the file:
@@
 P 12575 6475
 F 0 "R3" V 12775 6475 50  0000 C CNN
-F 1 "R" V 12675 6475 50  0000 C CNN
+F 1 "100K" V 12675 6475 50  0000 C CNN
 F 2 "Resistor_SMD:R_0201_0603Metric" V 12505 6475 50  0001 C CNN
 F 3 "~" H 12575 6475 50  0001 C CNN
@@
 P 10750 6425
 F 0 "R2" V 10950 6425 50  0000 C CNN
-F 1 "R" V 10850 6425 50  0000 C CNN
+F 1 "5.1K" V 10850 6425 50  0000 C CNN
 F 2 "Resistor_SMD:R_0201_0603Metric" V 10680 6425 50  0001 C CNN
 F 3 "~" H 10750 6425 50  0001 C CNN
@@
 P 10500 6150
 F 0 "R1" V 10700 6150 50  0000 C CNN
-F 1 "R" V 10600 6150 50  0000 C CNN
+F 1 "0" V 10600 6150 50  0000 C CNN
 F 2 "Resistor_SMD:R_0201_0603Metric" V 10430 6150 50  0001 C CNN
 F 3 "~" H 10500 6150 50  0001 C CNN
@@
 	1575 2425 1575 5225
 Wire Bus Line
-	6875 5225 9200 5225
-Wire Bus Line
 	5125 5225 6875 5225
 Wire Bus Line
@@
 Wire Wire Line
 	5525 10875 5525 10900
+Wire Bus Line
+	6875 5225 9200 5225
 $EndSCHEMATC
