File: KiCAD/matrixLED_array.sch (KiCad schematic (older format))
At the start: 28 parts, among them J10 Conn_01x12_Male, J11 Conn_01x12_Male, J12 Conn_01x12_Male, J13 Conn_01x12_Male, J14 Conn_01x12_Male, J15 Conn_01x12_Male, J16 Conn_01x12_Male, J17 Conn_01x12_Male, J2 Conn_01x12_Male, J3 Conn_01x12_Male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

Commit message: Datasheets folder
Parts:
- L1, L2, L3, L4, L5, L6, L7, L8: symbol myLedMatrix:LedMatrix_M -> driverDisplayLED-rescue:LedMatrix_M-myLedMatrix
Changed lines of the file:
@@
 $EndComp
 $Comp
-L myLedMatrix:LedMatrix_M L1
+L driverDisplayLED-rescue:LedMatrix_M-myLedMatrix L1
 U 1 1 66DEBDBB
 P 1565 2515
@@
 $EndComp
 $Comp
-L myLedMatrix:LedMatrix_M L3
+L driverDisplayLED-rescue:LedMatrix_M-myLedMatrix L3
 U 1 1 66F8FCA7
 P 3335 2515
@@
 $EndComp
 $Comp
-L myLedMatrix:LedMatrix_M L5
+L driverDisplayLED-rescue:LedMatrix_M-myLedMatrix L5
 U 1 1 67122D08
 P 5135 2515
@@
 $EndComp
 $Comp
-L myLedMatrix:LedMatrix_M L7
+L driverDisplayLED-rescue:LedMatrix_M-myLedMatrix L7
 U 1 1 6720A499
 P 6865 2515
@@
 $EndComp
 $Comp
-L myLedMatrix:LedMatrix_M L2
+L driverDisplayLED-rescue:LedMatrix_M-myLedMatrix L2
 U 1 1 675C996B
 P 1575 5075
@@
 $EndComp
 $Comp
-L myLedMatrix:LedMatrix_M L4
+L driverDisplayLED-rescue:LedMatrix_M-myLedMatrix L4
 U 1 1 675F6FE0
 P 3345 5075
@@
 $EndComp
 $Comp
-L myLedMatrix:LedMatrix_M L6
+L driverDisplayLED-rescue:LedMatrix_M-myLedMatrix L6
 U 1 1 6762E87D
 P 5145 5075
@@
 $EndComp
 $Comp
-L myLedMatrix:LedMatrix_M L8
+L driverDisplayLED-rescue:LedMatrix_M-myLedMatrix L8
 U 1 1 6766924C
 P 6865 5075
